File: MBC5 (Type A, FRAM)/mbc5_FRAM_typeA_1-1.kicad_pcb (KiCad board)
At the start: 2 copper layers, 53 x 62 mm, 12 parts, among them P1 GBC_CARTTAB, U10 74LVC1G332, U7 M29F160N, U8 MBC5, U9 FM18W08-SG

Commit message: Add files via upload
Parts:
- C21: value 100n -> 0.1u
Connections:
- net /PHI renamed /CLK
