File: MBC5 (Type A, FRAM)/mbc5_FRAM_typeA_1-1.kicad_sch (KiCad schematic)
At the start: 10 parts, among them P1 GBC_CARTTAB, U10 74LVC1G332, U7 M29F160N, U8 MBC5, U9 FM18W08-SG

Commit message: Add files via upload
Connections:
- net PHI renamed CLK
Other:
- company: (none) -> Mouse Bite Labs
- title: (none) -> Game Boy MBC5 Cartridge (FRAM, Type A)
Changed lines of the file:
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@@
 	(generator_version "8.0")
 	(paper "A4")
+	(title_block
+		(title "Game Boy MBC5 Cartridge (FRAM, Type A)")
+		(date "2024-12-28")
+		(rev "1.1")
+		(company "Mouse Bite Labs")
+	)
 	(bus_alias "GB_BUS"
 		(members "~{WR}" "~{RD}" "~{CS}" "A_{0}" "A_{1}" "A_{2}" "A_{3}" "A_{4}"
@@
 			"A_{14}" "A_{15}" "D_{0}" "D_{1}" "D_{2}" "D_{3}" "D_{4}" "D_{5}" "D_{6}"
 			"D_{7}" "RA_{14}" "RA_{15}" "RA_{16}" "RA_{17}" "RA_{18}" "RA_{19}" "RA_{20}"
-			"RA_{21}" "RA_{22}" "AA_{13}" "AA_{14}" "AA_{15}" "AA_{16}" "PHI"
+			"RA_{21}" "RA_{22}" "AA_{13}" "AA_{14}" "AA_{15}" "AA_{16}" "CLK"
 		)
 	)
@@
 		)
 	)
-	(label "PHI"
+	(label "CLK"
 		(at 144.78 127 0)
 		(fields_autoplaced yes)
@@
 		)
 	)
-	(label "PHI"
+	(label "CLK"
 		(at 35.56 34.29 180)
 		(fields_autoplaced yes)
