File: MBC3 (Type A, FRAM)/mbc3_FRAM_typeA_1-0.kicad_pcb (KiCad board)
At the start: 2 copper layers, 53 x 62 mm, 30 parts, among them P1 GBC_CARTTAB, Q3 2N7002, U10 74LVC1G332, U14 MM1134/MM1026, U15 TPS3613, U7 M29F160N, U8 MBC3, U9 FM18W08-SG, X3 XTAL-3.2X1.5

Commit message: Add files via upload
Parts:
- added G***: LOGO, LOGO, B.Cu at (148.5, 94.8)
